File: schematics/sonoff.kicad_pcb (KiCad board)
At the start: 2 copper layers, 49.9 x 43.1 mm, 17 parts, among them J1 Screw_Terminal_01x04, J2 Screw_Terminal_01x04, K1 Relay_SPDT, K2 Relay_SPDT, Q1 2N7000, Q2 2N7000, U1 ESP-01v090

Commit message: chore: improved design.
Parts:
- removed H3: MountingHole, MountingHole:MountingHole_4.5mm_Pad_TopBottom
- added J3: Conn_02x03_Odd_Even, Connector_PinHeader_2.54mm:PinHeader_2x03_P2.54mm_Vertical, F.Cu at (126.1, 112.3)
- added R3: R, Resistor_THT:R_Axial_DIN0207_L6.3mm_D2.5mm_P2.54mm_Vertical, F.Cu at (126.6, 107.3)
- J1: value Screw_Terminal_01x04 -> Screw_Terminal_01x06; footprint TerminalBlock:TerminalBlock_bornier-4_P5.08mm -> TerminalBlock:TerminalBlock_bornier-6_P5.08mm
- R1, R2: footprint Resistor_THT:R_Axial_DIN0207_L6.3mm_D2.5mm_P7.62mm_Horizontal -> Resistor_THT:R_Axial_DIN0207_L6.3mm_D2.5mm_P2.54mm_Vertical
- moved J1 55.5 mm to (179.3, 124.5), turned to 90 degrees
- moved H2 29.6 mm to (178.7, 89.8)
- moved D2 14.1 mm to (135.8, 104.3), turned to 180 degrees
- moved H1 13.4 mm to (135.3, 114.9)
- moved R2 10.7 mm to (126.6, 104.0), turned to 0 degrees
- moved R1 8.19 mm to (126.6, 100.7), turned to 0 degrees
- moved D1 6.74 mm to (135.8, 108.0), turned to 180 degrees
- moved C2 0.76 mm to (128.1, 95.8)
- moved K1 0.64 mm to (148.6, 124.3)
- moved K2 0.64 mm to (165.6, 124.3)
- moved J2 0.58 mm to (126.9, 123.3)
- moved Q1 0.25 mm to (134.5, 95.8)
- moved Q2 0.25 mm to (134.5, 100.6)
- moved C1 0.21 mm to (139.1, 86.7)
- renumbered Q2 to Q1, Q1 to Q2
Other:
- board size 49.9 x 43.1 mm -> 59.2 x 42.4 mm
- board text added: "## PINOUT ##"

Commit message: feat
Parts:
- removed the K2 at (165.6, 124.3)
- added JP1: SolderJumper_3_Open, Jumper:SolderJumper-3_P1.3mm_Open_Pad1.0x1.5mm, B.Cu at (170.9, 103.4)
- added JP2: SolderJumper_3_Open, Jumper:SolderJumper-3_P1.3mm_Open_Pad1.0x1.5mm, B.Cu at (167.1, 103.4)
- added JP3: SolderJumper_3_Open, Jumper:SolderJumper-3_P1.3mm_Open_Pad1.0x1.5mm, B.Cu at (163.2, 103.4)
- added JP4: SolderJumper_3_Open, Jumper:SolderJumper-3_P1.3mm_Open_Pad1.0x1.5mm, B.Cu at (159.4, 103.4)
- added JP5: SolderJumper_3_Open, Jumper:SolderJumper-3_P1.3mm_Open_Pad1.0x1.5mm, B.Cu at (155.6, 103.4)
- added JP6: SolderJumper_3_Open, Jumper:SolderJumper-3_P1.3mm_Open_Pad1.0x1.5mm, B.Cu at (151.7, 103.4)
- added JP7: SolderJumper_3_Open, Jumper:SolderJumper-3_P1.3mm_Open_Pad1.0x1.5mm, B.Cu at (147.9, 103.4)
- added JP8: SolderJumper_3_Open, Jumper:SolderJumper-3_P1.3mm_Open_Pad1.0x1.5mm, B.Cu at (144.1, 103.4)
- added K1: Relay_SPDT, Relay_THT:Relay_SPDT_Omron-G5LE-1, F.Cu at (165.6, 124.3)
- C1: value C -> 100nF
- C2: value C_Polarized -> 100uF
- R1, R2, R3: value R -> 10k
- U1: value ESP-01v090 -> ESP-01
- renumbered D2 to D1, D1 to D2, K1 to K2
Connections:
- C1 pad 1: unconnected-(C1-Pad1) -> +3.3V
- C1 pad 2: unconnected-(C1-Pad2) -> GND
- C2 pad 1: unconnected-(C2-Pad1) -> +3.3V
- C2 pad 2: unconnected-(C2-Pad2) -> GND
- D1 pad 1: unconnected-(D2-K-Pad1) -> +3.3V
- D1 pad 2: unconnected-(D2-A-Pad2) -> Net-(D1-A)
- D2 pad 1: unconnected-(D1-K-Pad1) -> +3.3V
- D2 pad 2: unconnected-(D1-A-Pad2) -> Net-(D2-A)
- J1 pad 1: unconnected-(J1-Pin_1-Pad1) -> /AC-L
- J1 pad 2: unconnected-(J1-Pin_2-Pad2) -> /AC-N
- J1 pad 3: unconnected-(J1-Pin_3-Pad3) -> /K1-1
- J1 pad 4: unconnected-(J1-Pin_4-Pad4) -> /K1-2
- J1 pad 5: unconnected-(J1-Pin_5-Pad5) -> /K2-1
- J1 pad 6: unconnected-(J1-Pin_6-Pad6) -> /K2-2
- J2 pad 1: unconnected-(J2-Pin_1-Pad1) -> GND
- J2 pad 2: unconnected-(J2-Pin_2-Pad2) -> /IN-2
- J2 pad 3: unconnected-(J2-Pin_3-Pad3) -> GND
- J2 pad 4: unconnected-(J2-Pin_4-Pad4) -> /IN-1
- J3 pad 1: unconnected-(J3-Pin_1-Pad1) -> /RST
- J3 pad 2: unconnected-(J3-Pin_2-Pad2) -> /GPIO0
- J3 pad 3: unconnected-(J3-Pin_3-Pad3) -> /GPIO3
- J3 pad 4: unconnected-(J3-Pin_4-Pad4) -> /GPIO1
- J3 pad 5: unconnected-(J3-Pin_5-Pad5) -> +3.3V
- J3 pad 6: unconnected-(J3-Pin_6-Pad6) -> GND
- K2 pad 1: (no net) -> /K2-1
- K2 pad 2: (no net) -> Net-(D2-A)
- K2 pad 3: (no net) -> /K2-2
- K2 pad 4: (no net) -> unconnected-(K2-Pad4)
- K2 pad 5: (no net) -> +3.3V
- PS1 pad 1: unconnected-(PS1-AC/L-Pad1) -> /AC-L
- PS1 pad 2: unconnected-(PS1-AC/N-Pad2) -> /AC-N
- PS1 pad 3: unconnected-(PS1--Vout-Pad3) -> GND
- PS1 pad 4: unconnected-(PS1-+Vout-Pad4) -> +3.3V
- Q1 pad 1: unconnected-(Q1-S-Pad1) -> GND
- Q1 pad 2: unconnected-(Q1-G-Pad2) -> /OUT-1
- Q1 pad 3: unconnected-(Q1-D-Pad3) -> Net-(D1-A)
- Q2 pad 1: unconnected-(Q2-S-Pad1) -> GND
- Q2 pad 2: unconnected-(Q2-G-Pad2) -> /OUT-2
- Q2 pad 3: unconnected-(Q2-D-Pad3) -> Net-(D2-A)
- R1 pad 1: unconnected-(R1-Pad1) -> +3.3V
- R1 pad 2: unconnected-(R1-Pad2) -> /GPIO0
- R2 pad 1: unconnected-(R2-Pad1) -> +3.3V
- R2 pad 2: unconnected-(R2-Pad2) -> /GPIO2
- R3 pad 1: unconnected-(R3-Pad1) -> +3.3V
- R3 pad 2: unconnected-(R3-Pad2) -> /RST
- U1 pad 1: unconnected-(U1-UTXD-Pad1) -> /GPIO1
- U1 pad 2: unconnected-(U1-GND-Pad2) -> GND
- U1 pad 3: unconnected-(U1-CH_PD-Pad3) -> +3.3V
- U1 pad 4: unconnected-(U1-GPIO2-Pad4) -> /GPIO2
- U1 pad 5: unconnected-(U1-RST-Pad5) -> /RST
- U1 pad 6: unconnected-(U1-GPIO0-Pad6) -> /GPIO0
- U1 pad 7: unconnected-(U1-VCC-Pad7) -> +3.3V
- U1 pad 8: unconnected-(U1-URXD-Pad8) -> /GPIO3
Routing:
- net +3.3V: track 0.00 -> 134.7 mm
- net /GPIO1: track 0.00 -> 85.2 mm, vias 0 -> 2
- net /GPIO0: track 0.00 -> 69.6 mm, vias 0 -> 2
- net Net-(D1-A): track 0.00 -> 67.5 mm, vias 0 -> 3
- net /GPIO3: track 0.00 -> 64.6 mm, vias 0 -> 2
- net /IN-2: track 0.00 -> 62.6 mm, vias 0 -> 4
- net /IN-1: track 0.00 -> 54.3 mm, vias 0 -> 4
- net /GPIO2: track 0.00 -> 48.5 mm, vias 0 -> 1
- net /K2-1: track 0.00 -> 48.4 mm
- net /OUT-1: track 0.00 -> 46.6 mm, vias 0 -> 4
- net /OUT-2: track 0.00 -> 43.5 mm, vias 0 -> 4
- net /AC-L: track 0.00 -> 41.7 mm
- net /AC-N: track 0.00 -> 40.8 mm
- net Net-(D2-A): track 0.00 -> 39.7 mm, vias 0 -> 1
- net /RST: track 0.00 -> 33.8 mm
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- added copper zone on B.Cu, net GND
Other:
- board text added: "D0"
- board text added: "D1"
- board text added: "D2"
- board text added: "D3"
- board text added: "IN-1"
- board text added: "IN-2"
- board text added: "OUT-1"
- board text added: "OUT-2"

Commit message: !feat: first rev2 release
Parts:
- added G***: LOGO, LOGO, B.Cu at (110.3, 49.3)
- U1: value ESP-01 -> ESP-01_2x04
- moved JP8 63.2 mm to (96.9, 61.2)
- moved D2 63.2 mm to (88.7, 65.8)
- moved J3 63.2 mm to (79.0, 70.1)
- moved JP1 63.2 mm to (123.8, 61.2)
- moved JP2 63.2 mm to (120.0, 61.2)
- moved JP5 63.2 mm to (108.5, 61.2)
- moved JP6 63.2 mm to (104.6, 61.2)
- moved R1 63.2 mm to (79.5, 58.5)
- moved R2 63.2 mm to (79.5, 61.8)
- moved R3 63.2 mm to (79.5, 65.2)
- moved U1 63.2 mm to (88.6, 45.0)
- moved C1 63.2 mm to (91.9, 44.5)
- moved C2 63.2 mm to (81.0, 53.6)
- moved D1 63.2 mm to (88.7, 62.1)
- moved H1 63.2 mm to (88.1, 72.8)
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Routing:
- net /AC-N: track 40.8 -> 42.8 mm
- net /AC-L: track 41.7 -> 43.5 mm
- net /K2-2: track 30.6 -> 32.3 mm
- net +3.3V: track 134.7 -> 133.9 mm
Other:
- board size 59.2 x 42.4 mm -> 59.2 x 42.9 mm
- board text added: "-"
- board text added: "AC-L"
- board text added: "AC-N"
- board text added: "DIY ESP-01 Sonoff Davide Scalisi Rev. 2.0"
- board text added: "K1-1"
- board text added: "K1-2"
- board text added: "K2-1"
- board text added: "K2-2"
- board text removed: "## LOGO ##"
- board text removed: "## PINOUT ##"

Commit message: feat: added "JLCJLCJLCJLC" to the back of the PCB.
Other:
- board text added: "JLCJLCJLCJLC"
Changed lines of the file:
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@@
+		)
+	)
+	(gr_text "JLCJLCJLCJLC"
+		(at 129.54 84.074 0)
+		(layer "B.SilkS")
+		(effects
+			(font
+				(size 0.8 0.8)
+				(thickness 0.15)
+				(bold yes)
+			)
+			(justify left bottom mirror)
 		)
 	)
